Commit message: Improve LiDAR scan accuracy with exact-mesh collision shapes
Replace single bounding-box collision on shelves and forklift with
per-triangle BVH collision (GEOM_FORCE_CONCAVE_TRIMESH). Rays now
resolve actual mesh geometry — shelf uprights, board levels, and
forklift forks/mast/cab — instead of a solid parallelepiped hull.

world.py switches from loadURDF to programmatic createMultiBody so the
OBJ files can be used directly as concave trimesh collision shapes.
URDF files are updated with compound-box fallback geometry for reference.

File: assets/forklift/forklift.urdf (robot description, URDF)
Before this commit: robot forklift, 1 links, 0 joints
Links:
- link base_link: geometry collision box size=0.22 1.24 2.50; collision box size=0.78 1.24 0.25

File: assets/shelf/shelf_bay.urdf (robot description, URDF)
Before this commit: robot shelf_bay, 1 links, 0 joints
Links:
- link base_link: geometry collision box size=0.04 1.04 2.50; collision box size=0.06 0.06 2.50
